Commit message: el paquete bringup ya funciona con phantomx_pincher.launch.py, tambien funcion commander_template.cpp

File: phantom_ws/src/phantomx_pincher_description/urdf/phantomx_pincher.urdf.xacro (robot description, xacro)
@@ -1,5 +1,5 @@
 <?xml version="1.0"?>
 <!-- URDF for PhantomX Pincher Robot Arm -->
-<robot xmlns:xacro="http://wiki.ros.org/xacro" name="$(arg name)">
+<robot xmlns:xacro="http://wiki.ros.org/xacro" name="phantomx_pincher">
   <!--                   -->
   <!-- Imported elements -->
@@ -25,8 +25,10 @@
   <!-- The ros2_control plugin that should be loaded for the manipulator ('fake', 'ign', 'real' or custom) -->
   <xacro:arg name="ros2_control_plugin" default="fake"/>
-  <!-- The output control command interface provided by ros2_control ('position', 'velocity', 'effort' or certain combinations 'position,velocity') -->
+  <!-- The output control command interface provided by ros2_control
+       ('position', 'velocity', 'effort' or combinations like 'position,velocity') -->
   <xacro:arg name="ros2_control_command_interface" default="position"/>
   <!-- The filepath to parameters of ROS 2 controllers -->
-  <xacro:arg name="ros2_controller_parameters" default="$(find phantomx_pincher_moveit_config)/config/controllers_$(arg ros2_control_command_interface).yaml"/>
+  <xacro:arg name="ros2_controller_parameters"
+             default="$(find phantomx_pincher_moveit_config)/config/controllers_$(arg ros2_control_command_interface).yaml"/>
   <!-- Flag to enable mimicking of the finger joints -->
   <xacro:arg name="mimic_finger_joints" default="false"/>
@@ -49,5 +51,5 @@
     <parent link="$(arg prefix)${base_link}"/>
     <!-- Root of the kit defined in kit.xacro -->
-    <child  link="world_link"/>
+    <child link="world_link"/>
     <origin xyz="0 0 0" rpy="0 0 0"/>
   </joint>
@@ -57,12 +59,6 @@
     <parent link="caseBaseRobot_link"/>
     <!-- Child: base link of the PhantomX arm -->
-    <child  link="$(arg prefix)arm_base_link"/>
-    <!--
-      TODO: adjust xyz and rpy so that the arm base coincides
-      with the mounting holes on caseBaseRobot_link.
-      Start with zeros and tune:
-        xyz = "x y z"
-        rpy = "roll pitch yaw"
-    -->
+    <child link="$(arg prefix)arm_base_link"/>
+    <!-- Pose of the arm base relative to the kit (tuned in original repo) -->
     <origin xyz="0.01325 0 0.016" rpy="0 0 0"/>
   </joint>
@@ -77,27 +73,28 @@
       mimic_finger_joints="$(arg mimic_finger_joints)"
       gazebo_preserve_fixed_joint="$(arg gazebo_preserve_fixed_joint)"/>
-  <!--       -->
-  <!-- Robot -->
-  <!--       -->
-  <!-- Base link that can be used for fixing the robot to the world
-  <xacro:phantomx_pincher_dummy_link link_name="$(arg prefix)${base_link}" gazebo_preserve_fixed_joint="$(arg gazebo_preserve_fixed_joint)"/>
-  <joint name="$(arg prefix)${base_link}_joint" type="fixed">
-    <parent link="$(arg prefix)${base_link}"/>
-    <child link="$(arg prefix)task_board_link"/>
-  </joint>
-   -->
-  <!-- Mount
-  <xacro:task_board prefix="$(arg prefix)" child="task_board_mount_link" collision="$(arg collision)" gazebo_preserve_fixed_joint="$(arg gazebo_preserve_fixed_joint)"/>
-  <xacro:task_board_mount prefix="$(arg prefix)" child="base_mount_link" collision="$(arg collision)" gazebo_preserve_fixed_joint="$(arg gazebo_preserve_fixed_joint)"/>
-  <xacro:base_mount prefix="$(arg prefix)" child="arm_base_link" collision="$(arg collision)" gazebo_preserve_fixed_joint="$(arg gazebo_preserve_fixed_joint)"/>
+  <!-- Example environment / mounting macros (kept commented out) -->
+  <!--
+  <xacro:task_board
+      prefix="$(arg prefix)"
+      child="task_board_mount_link"
+      collision="$(arg collision)"
+      gazebo_preserve_fixed_joint="$(arg gazebo_preserve_fixed_joint)"/>
+  <xacro:task_board_mount
+      prefix="$(arg prefix)"
+      child="base_mount_link"
+      collision="$(arg collision)"
+      gazebo_preserve_fixed_joint="$(arg gazebo_preserve_fixed_joint)"/>
+  <xacro:base_mount
+      prefix="$(arg prefix)"
+      child="arm_base_link"
+      collision="$(arg collision)"
+      gazebo_preserve_fixed_joint="$(arg gazebo_preserve_fixed_joint)"/>
   -->
-  <!-- Arm
-  <xacro:phantomx_pincher prefix="$(arg prefix)" base_link="arm_base_link" collision="$(arg collision)" ros2_control="$(arg ros2_control)" ros2_control_plugin="$(arg ros2_control_plugin)" ros2_control_command_interface="$(arg ros2_control_command_interface)" mimic_finger_joints="$(arg mimic_finger_joints)" gazebo_preserve_fixed_joint="$(arg gazebo_preserve_fixed_joint)"/>
-  -->
-  <!-- Gazebo - ROS 2 control (Ignition) -->
+  <!-- Gazebo - ROS 2 control (Ignition)
   <xacro:if value="$(arg ros2_control)">
     <xacro:if value="${'ign' in '$(arg ros2_control_plugin)' or 'gz' in '$(arg ros2_control_plugin)'}">
-      <xacro:ign_ros2_control controller_parameters="$(find phantomx_pincher_moveit_config)/config/controllers_$(arg ros2_control_command_interface).yaml"/>
+      <xacro:ign_ros2_control controller_parameters="$(arg ros2_controller_parameters)"/>
     </xacro:if>
   </xacro:if>
+  -->
 </robot>
