Commit message: Update

File: phantom_ws/src/phantomx_pincher_description/urdf/phantomx_pincher.urdf (robot description, URDF)
Before this commit: robot phantomx_pincher, 35 links, 34 joints
Links:
- added link canastilla_link; collision box size=0.02 0.36000000000000004 0.1855; collision box size=0.02 0.36000000000000004 0.1855
- added link ensambleSoporteCamara_link; collision box size=0.04 0.04 0.30; visual mesh filename=package://phantomx_pincher_description/meshes/STL/ensambleS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 scale=0.001 0.001 0.001
Joints:
- added joint base_canastilla_joint: type fixed, parent baseFija_link, child canastilla_link, origin xyz=0.155 0 -0.0145 rpy=0 0 0
- added joint base_ensambleSoporteCamara_joint: type fixed, parent baseFija_link, child ensambleSoporteCamara_link, origin xyz=0.26 0 0.00 rpy=0 0 -1.5707963267948966
